File: lamp-controller.kicad_pcb (KiCad board)
At the start: 0 parts

Commit message: Layout
Parts:
- added C1: 1u, Capacitor_SMD:C_0805_2012Metric_Pad1.18x1.45mm_HandSolder, F.Cu at (135.8, 75.0)
- added C2: 10u 16v, Capacitor_THT:CP_Radial_D4.0mm_P2.00mm, F.Cu at (135.7, 86.3)
- added C3: 1u, Capacitor_SMD:C_0805_2012Metric_Pad1.18x1.45mm_HandSolder, F.Cu at (141.5, 75.1)
- added C4: 1u, Capacitor_SMD:C_0805_2012Metric_Pad1.18x1.45mm_HandSolder, F.Cu at (140.2, 87.5)
- added C5: 0u1, Capacitor_SMD:C_0805_2012Metric_Pad1.18x1.45mm_HandSolder, F.Cu at (140.6, 80.0)
- added C6: 0u1, Capacitor_SMD:C_0805_2012Metric_Pad1.18x1.45mm_HandSolder, F.Cu at (140.6, 82.0)
- added C7: 0u1, Capacitor_SMD:C_0805_2012Metric_Pad1.18x1.45mm_HandSolder, F.Cu at (147.5, 85.9)
- added C8: 10u 16v, Capacitor_THT:CP_Radial_D4.0mm_P2.00mm, F.Cu at (161.0, 84.5)
- added H1: MountingHole_Pad, MountingHole:MountingHole_2.2mm_M2_DIN965_Pad, F.Cu at (132.6, 72.2)
- added H2: MountingHole_Pad, MountingHole:MountingHole_2.2mm_M2_DIN965_Pad, F.Cu at (132.6, 92.5)
- added H3: MountingHole_Pad, MountingHole:MountingHole_2.2mm_M2_DIN965_Pad, F.Cu at (147.4, 92.5)
- added J1: Conn_01x02_Pin, Connector_PinHeader_2.54mm:PinHeader_1x02_P2.54mm_Vertical, F.Cu at (131.5, 80.5)
- added J2: Conn_ARM_JTAG_SWD_10, Connector_PinHeader_1.27mm:PinHeader_2x05_P1.27mm_Vertical, F.Cu at (149.3, 74.5)
- added J3: Conn_01x04_Socket, Connector_PinHeader_2.54mm:PinHeader_1x04_P2.54mm_Vertical, F.Cu at (162.6, 71.1)
- added J4: Conn_01x03_Socket, Connector_PinHeader_2.54mm:PinHeader_1x03_P2.54mm_Vertical, F.Cu at (162.6, 88.9)
- added J5: Conn_01x03_Male, Connector_PinHeader_1.00mm:PinHeader_1x03_P1.00mm_Vertical, F.Cu at (141.9, 94.8)
- added Q1: DMN2053UVT, Package_TO_SOT_SMD:TSOT-23-6, F.Cu at (157.7, 79.0)
- added Q2: DMN2053UVT, Package_TO_SOT_SMD:TSOT-23-6, F.Cu at (157.8, 73.0)
- added R1: 10k, Resistor_SMD:R_0603_1608Metric_Pad0.98x0.95mm_HandSolder, F.Cu at (140.8, 78.1)
- added R2: 10k, Resistor_SMD:R_0603_1608Metric_Pad0.98x0.95mm_HandSolder, F.Cu at (155.2, 82.9)
- added R3: 10k, Resistor_SMD:R_0603_1608Metric_Pad0.98x0.95mm_HandSolder, F.Cu at (157.0, 82.9)
- added R4: 10k, Resistor_SMD:R_0603_1608Metric_Pad0.98x0.95mm_HandSolder, F.Cu at (153.9, 72.1)
- added R5: 10k, Resistor_SMD:R_0603_1608Metric_Pad0.98x0.95mm_HandSolder, F.Cu at (147.5, 89.2)
- added R6: 10k, Resistor_SMD:R_0603_1608Metric_Pad0.98x0.95mm_HandSolder, F.Cu at (153.9, 74.4)
- added R7: 100R, Resistor_SMD:R_0603_1608Metric_Pad0.98x0.95mm_HandSolder, F.Cu at (147.5, 87.7)
- added R8: 10k, Resistor_SMD:R_0603_1608Metric_Pad0.98x0.95mm_HandSolder, F.Cu at (153.9, 78.1)
- added RV1: 100k, Connector_PinHeader_1.27mm:PinHeader_1x03_P1.27mm_Vertical, F.Cu at (151.4, 91.1)
- added RV2: 100k, Connector_PinHeader_1.27mm:PinHeader_1x03_P1.27mm_Vertical, F.Cu at (154.5, 91.1)
- added RV3: 100k, Connector_PinHeader_1.27mm:PinHeader_1x03_P1.27mm_Vertical, F.Cu at (157.6, 91.1)
- added SW1: SW_SPST, Connector_PinHeader_2.54mm:PinHeader_1x02_P2.54mm_Vertical, F.Cu at (135.8, 80.5)
- added SW2: SW_Push, Connector_PinHeader_1.27mm:PinHeader_1x02_P1.27mm_Vertical, F.Cu at (143.9, 85.8)
- added U1: MIC5365-3.3YC5, Package_TO_SOT_SMD:SOT-353_SC-70-5, F.Cu at (138.7, 74.6)
- added U2: STM32L010F4Px, Package_SO:TSSOP-20_4.4x6.5mm_P0.65mm, F.Cu at (146.7, 80.9)
Routing:
- net +5V: track 0.00 -> 67.8 mm, vias 0 -> 3
- net +3V3: track 0.00 -> 50.0 mm, vias 0 -> 6
- net GND: track 0.00 -> 23.2 mm, vias 0 -> 55
- net /A_Pot: track 0.00 -> 16.2 mm
- net /PxCtrl: track 0.00 -> 16.0 mm
- net /C_Pot: track 0.00 -> 14.7 mm
- net /LPUART1_TX: track 0.00 -> 13.5 mm
- net /LPUART1_RX: track 0.00 -> 13.0 mm
- net /A: track 0.00 -> 12.0 mm
- net /B_Pot: track 0.00 -> 11.4 mm
- net /PxCtrlLv: track 0.00 -> 11.2 mm
- net /B: track 0.00 -> 10.4 mm
- net /C: track 0.00 -> 9.88 mm, vias 0 -> 2
- net /Button: track 0.00 -> 9.22 mm, vias 0 -> 2
- net /rst: track 0.00 -> 7.71 mm
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- added copper zone on B.Cu, net +5V
- added copper zone on F.Cu, net +5V
- added copper zone on B.Cu, net GND
- added copper zone on F.Cu, net GND
Other:
- board outline added: 34.9 x 26.5 mm
- copper layers 0 -> 2
- board text added: "JLCJLCJLCJLC"
- board text added: "Simple lamp controller V1.0a D. Miall 2023"
