File: lamp-controller.kicad_sch (KiCad schematic)
At the start: 9 parts, among them J1 Conn_01x02_Pin, J2 Conn_ARM_JTAG_SWD_10, J3 Conn_01x04_Socket, U1 STM32L010F4Px, U2 MIC5365-3.3YC5

Commit message: Layout
Parts:
- removed C1: 10u 16v, Capacitor_SMD:CP_Elec_4x4.5, symbol Device:C_Polarized
- removed C2: 1u, Capacitor_SMD:C_0805_2012Metric_Pad1.18x1.45mm_HandSolder, symbol Device:C
- removed U1: STM32L010F4Px, Package_SO:TSSOP-20_4.4x6.5mm_P0.65mm, symbol MCU_ST_STM32L0:STM32L010F4Px
- added C2, C8: 10u 16v, Capacitor_THT:CP_Radial_D4.0mm_P2.00mm, symbol Device:C_Polarized
- added C4: 1u, Capacitor_SMD:C_0805_2012Metric_Pad1.18x1.45mm_HandSolder, symbol Device:C
- added C5, C6, C7: 0u1, Capacitor_SMD:C_0805_2012Metric_Pad1.18x1.45mm_HandSolder, symbol Device:C
- added H1, H2, H3: MountingHole_Pad, MountingHole:MountingHole_2.2mm_M2_DIN965_Pad, symbol Mechanical:MountingHole_Pad
- added J4: Conn_01x03_Socket, Connector_PinHeader_2.54mm:PinHeader_1x03_P2.54mm_Vertical, symbol Connector:Conn_01x03_Socket
- added J5: Conn_01x03_Male, Connector_PinHeader_1.00mm:PinHeader_1x03_P1.00mm_Vertical, symbol Connector:Conn_01x03_Male
- added Q1, Q2: DMN2053UVT, Package_TO_SOT_SMD:TSOT-23-6, symbol kicad_global_library:DMN2053UVT
- added R1, R2, R3, R4, R5, R6, R8: 10k, Resistor_SMD:R_0603_1608Metric_Pad0.98x0.95mm_HandSolder, symbol Device:R
- added R7: 100R, Resistor_SMD:R_0603_1608Metric_Pad0.98x0.95mm_HandSolder, symbol Device:R
- added RV1, RV2, RV3: 100k, Connector_PinHeader_1.27mm:PinHeader_1x03_P1.27mm_Vertical, symbol Device:R_Potentiometer
- added SW1: SW_SPST, Connector_PinHeader_2.54mm:PinHeader_1x02_P2.54mm_Vertical, symbol Switch:SW_SPST
- added SW2: SW_Push, Connector_PinHeader_1.27mm:PinHeader_1x02_P1.27mm_Vertical, symbol Switch:SW_Push
- added U2: STM32L010F4Px, Package_SO:TSSOP-20_4.4x6.5mm_P0.65mm, symbol MCU_ST_STM32L0:STM32L010F4Px
- J1: footprint (none) -> Connector_PinHeader_2.54mm:PinHeader_1x02_P2.54mm_Vertical
- J2: footprint (none) -> Connector_PinHeader_1.27mm:PinHeader_2x05_P1.27mm_Vertical
- J3: footprint (none) -> Connector_PinHeader_2.54mm:PinHeader_1x04_P2.54mm_Vertical
- renumbered C4 to C1, U2 to U1
Connections:
- net +3V3: now also C6.1, Q1.3 (G), R2.1, R5.1, RV1.1, RV2.1, RV3.1, U2.16 (VDD), U2.5 (VDDA)
- net +5V: now also J3.4 (Pin_4), C2.1, C4.1, C8.1, J4.1 (Pin_1), R3.1, SW1.2 (B); no longer J1.1 (Pin_1), J3.1 (Pin_1)
- net GND: now also J2.3 (GND), J2.5 (GND), C2.2, C4.2, C5.2, C6.2, C7.2, C8.2, H1.1, H2.1, H3.1, J4.3 (Pin_3), J5.3 (Pin_3), Q1.5 (S), Q2.2 (S), Q2.5 (S), R1.2, R4.2, R6.2, R8.2, RV1.3, RV2.3, RV3.3, SW2.1, U2.15 (VSS)
- net 3v3: now reaches J2.1 (VTref)
- net rst: now reaches J2.10 (~{RESET})
- net rst: now also C5.1, U2.4 (NRST)
- net swdio: now reaches J2.2 (SWDIO/TMS)
- net swdio: now also U2.19 (PA13)
- net swclk: now reaches J2.4 (SWDCLK/TCK)
- net swclk: now also U2.20 (PA14)
- net B_o: now reaches J3.2 (Pin_2)
- net B_o: now also Q2.4 (D)
- net C_o: now reaches J3.3 (Pin_3)
- net C_o: now also Q1.6 (D)
- new net: R5.2, R7.1, SW2.2
- new net: R1.1, U2.1 (PB9)
- new net 5Vin: J1.1 (Pin_1), SW1.1 (A)
- new net A: Q2.1 (G), R4.1, U2.18 (PA10)
- new net A_Pot: RV1.2, U2.10 (PA4)
- new net A_o: J3.1 (Pin_1), Q2.6 (D)
- new net B: Q2.3 (G), R6.1, U2.17 (PA9)
- new net B_Pot: RV2.2, U2.11 (PA5)
- new net Button: C7.1, R7.2, U2.7 (PA1)
- new net C: Q1.1 (G), R8.1, U2.13 (PA7)
- new net C_Pot: RV3.2, U2.12 (PA6)
- new net LPUART1_RX: J5.2 (Pin_2), U2.9 (PA3)
- new net LPUART1_TX: J5.1 (Pin_1), U2.8 (PA2)
- new net PxCtrl: J4.2 (Pin_2), Q1.4 (D), R3.2
- new net PxCtrlLv: Q1.2 (S), R2.2, U2.14 (PB1)
- no-connect marks 0 -> 5
Other:
- note added: "No on-board current regulation. Make sure to add resistors to the strings!"
- note added: "STM32L011F4 is pin-compatible"
- note added: "Simple LED Lamp controller"
- note added: "The DMN2053UVT can pass 4.2A max Which is much more than most 5V supplies that are likely to be used could supply."
- note added: "Three channel LED drive. Intended to drive paralleled strings."
- note added: "UART"
- note added: "WS2812B String"
- moved on the sheet: J3

Commit message: RP2040 Version
Parts:
- removed C5: 0u1, Capacitor_SMD:C_0805_2012Metric_Pad1.18x1.45mm_HandSolder, symbol Device:C
- removed J1: Conn_01x02_Pin, Connector_PinHeader_2.54mm:PinHeader_1x02_P2.54mm_Vertical, symbol Connector:Conn_01x02_Pin
- removed J3: Conn_01x04_Socket, Connector_PinHeader_2.54mm:PinHeader_1x04_P2.54mm_Vertical, symbol Connector:Conn_01x04_Socket
- removed R1: 10k, Resistor_SMD:R_0603_1608Metric_Pad0.98x0.95mm_HandSolder, symbol Device:R
- removed U1: MIC5365-3.3YC5, Package_TO_SOT_SMD:SOT-353_SC-70-5, symbol Regulator_Linear:MIC5365-3.3YC5
- removed U2: STM32L010F4Px, Package_SO:TSSOP-20_4.4x6.5mm_P0.65mm, symbol MCU_ST_STM32L0:STM32L010F4Px
- added C10, C11, C12, C13, C14, C15, C16, C7, C8, C9: 100n, Capacitor_SMD:C_0603_1608Metric_Pad1.08x0.95mm_HandSolder, symbol Device:C
- added C17, C23, C24: 0u1, Capacitor_SMD:C_0603_1608Metric_Pad1.08x0.95mm_HandSolder, symbol Device:C
- added C19: 10p, Capacitor_SMD:C_0603_1608Metric_Pad1.08x0.95mm_HandSolder, symbol Device:C
- added C20, C21: 27p, Capacitor_SMD:C_0603_1608Metric_Pad1.08x0.95mm_HandSolder, symbol Device:C
- added C5: 10u 16v, Capacitor_THT:CP_Radial_D4.0mm_P2.00mm, symbol Device:C_Polarized
- added H4: MountingHole_Pad, MountingHole:MountingHole_2.2mm_M2_DIN965_Pad, symbol Mechanical:MountingHole_Pad
- added J1: Conn_02x06_Odd_Even, Connector_PinHeader_2.00mm:PinHeader_2x06_P2.00mm_Vertical, symbol Connector_Generic:Conn_02x06_Odd_Even
- added J2: Conn_02x05_Odd_Even, Connector_PinHeader_2.54mm:PinHeader_2x05_P2.54mm_Vertical, symbol Connector_Generic:Conn_02x05_Odd_Even
- added J7: Conn_01x04_Socket, Connector_PinHeader_2.54mm:PinHeader_1x04_P2.54mm_Vertical, symbol Connector:Conn_01x04_Socket
- added J8: USB_B_Micro, Connector_USB:USB_Micro-B_Amphenol_10103594-0001LF_Horizontal, symbol Connector:USB_B_Micro
- added JP1: SolderJumper_2_Open, Jumper:SolderJumper-2_P1.3mm_Open_RoundedPad1.0x1.5mm, symbol Jumper:SolderJumper_2_Open
- added Q3: DMN2053UVT, Package_TO_SOT_SMD:TSOT-23-6, symbol kicad_global_library:DMN2053UVT
- added R11, R12, R4, R5: 10k, Resistor_SMD:R_0603_1608Metric_Pad0.98x0.95mm_HandSolder, symbol Device:R
- added R13: 1k3, Resistor_SMD:R_0603_1608Metric_Pad0.98x0.95mm_HandSolder, symbol Device:R
- added R15, R16: 100R, Resistor_SMD:R_0603_1608Metric_Pad0.98x0.95mm_HandSolder, symbol Device:R
- added R6, R7: 27R, Resistor_SMD:R_0603_1608Metric_Pad0.98x0.95mm_HandSolder, symbol Device:R
- added SW3, SW4: SW_Push, Connector_PinHeader_1.27mm:PinHeader_1x02_P1.27mm_Vertical, symbol Switch:SW_Push
- added U1: AP2202K-3.3TRG1, Package_TO_SOT_SMD:SOT-23-5, symbol kicad_global_library:AP2202K
- added U2: W25Q16JVSS, Package_SO:SOIC-8_5.275x5.275mm_P1.27mm, symbol kicad_global_library:W25Q16JVSS
- added U3: RP2040, Package_DFN_QFN:QFN-56-1EP_7x7mm_P0.4mm_EP3.2x3.2mm, symbol kicad_global_library:RP2040
- added Y1: RH100-12.000-18-2030-TR, Crystal:Crystal_SMD_3225-4Pin_3.2x2.5mm, symbol Device:Crystal_GND24
- C1, C4: footprint Capacitor_SMD:C_0805_2012Metric_Pad1.18x1.45mm_HandSolder -> Capacitor_SMD:C_0603_1608Metric_Pad1.08x0.95mm_HandSolder
- C2: renamed from C3; footprint Capacitor_SMD:C_0805_2012Metric_Pad1.18x1.45mm_HandSolder -> Capacitor_SMD:C_0603_1608Metric_Pad1.08x0.95mm_HandSolder
- C22: renamed from C7; footprint Capacitor_SMD:C_0805_2012Metric_Pad1.18x1.45mm_HandSolder -> Capacitor_SMD:C_0603_1608Metric_Pad1.08x0.95mm_HandSolder
- C6: value 0u1 -> 100n; footprint Capacitor_SMD:C_0805_2012Metric_Pad1.18x1.45mm_HandSolder -> Capacitor_SMD:C_0603_1608Metric_Pad1.08x0.95mm_HandSolder
- renumbered C8 to C18, C2 to C3, J4 to J3, J2 to J5, J5 to J6, R8 to R1, R5 to R10, R7 to R14, R4 to R2, R6 to R3, R3 to R8, R2 to R9, RV3 to RV1, RV1 to RV3
Connections:
- net 3v3 is gone; now on net +3V3: J5.1 (VTref)
- net +3V3: now also C10.2, C11.2, C12.2, C13.2, C14.2, C15.2, C16.2, C17.1, C9.2, R11.1, R12.1, U1.5 (VOUT), U2.8 (VCC), U3.1 (IOVDD), U3.10 (IOVDD), U3.22 (IOVDD), U3.33 (IOVDD), U3.42 (IOVDD), U3.43 (ADC_AVDD), U3.44 (VREG_IN), U3.48 (USB_VDD), U3.49 (IOVDD); no longer C6.1
- net +5V: now also C5.1, J2.10 (Pin_10), J2.2 (Pin_2), J2.4 (Pin_4), J2.6 (Pin_6), J2.8 (Pin_8), U1.1 (VIN), U1.3 (EN)
- net 5Vin: now also J7.1 (Pin_1), J8.1 (VBUS)
- net A: now also R1.1, U3.4 (GPIO2); no longer R2.1
- net A_o: now also J2.1 (Pin_1)
- net B: now also R2.1, U3.6 (GPIO4); no longer R3.1
- net B_o: now also J2.3 (Pin_3)
- net C: now also R3.1, Q3.1 (G), U3.8 (GPIO6); no longer Q1.1 (G), R1.1
- net C_o: now also J2.5 (Pin_5), Q3.6 (D); no longer Q1.6 (D)
- net GND: now also C6.1, C10.1, C11.1, C12.1, C13.1, C14.1, C15.1, C16.1, C17.2, C19.2, C20.2, C21.2, C23.2, C24.2, C5.2, C7.1, C8.1, C9.1, H4.1, J1.1 (Pin_1), J1.11 (Pin_11), J1.3 (Pin_3), J1.5 (Pin_5), J1.7 (Pin_7), J1.9 (Pin_9), J7.4 (Pin_4), J8.5 (GND), JP1.1 (A), Q3.2 (S), Q3.5 (S), R4.2, R5.2, SW3.1, SW4.1, U1.2 (GND), U2.4 (GND), U3.19 (TESTEN), U3.57 (GND), Y1.2, Y1.4; no longer C6.2
- net PxCtrlLv: now also U3.5 (GPIO3)
- net rst: now also U3.26 (RUN)
- net swclk: now also U3.24 (SWCLK)
- net swdio: now also U3.25 (SWD)
- net A_Pot renamed Pot_1
- net Pot_1: now also U3.38 (GPIO26_ADC0)
- net B_Pot renamed Pot_2
- net Pot_2: now also U3.39 (GPIO27_ADC1)
- net Button renamed Button_1
- net Button_1: now also U3.7 (GPIO5)
- net C_Pot renamed Pot_3
- net Pot_3: now also U3.40 (GPIO28_ADC2)
- net LPUART1_RX renamed UART0_RX
- net UART0_RX: now also U3.3 (GPIO1)
- net LPUART1_TX renamed UART0_TX
- net UART0_TX: now also U3.2 (GPIO0)
- new net: J1.10 (Pin_10), U3.18 (GPIO15)
- new net: J1.2 (Pin_2), U3.14 (GPIO11)
- new net: J1.4 (Pin_4), U3.15 (GPIO12)
- new net: J1.6 (Pin_6), U3.16 (GPIO13)
- new net: J1.8 (Pin_8), U3.17 (GPIO14)
- new net: R6.2, U3.47 (USB_DP)
- new net: R7.2, U3.46 (USB_DM)
- new net: C20.1, R13.2, Y1.1
- new net: C19.1, J8.6 (Shield)
- new net: R11.2, R15.1, SW3.2
- new net: R12.2, R16.1, SW4.2
- new net +1V1: C6.2, C7.2, C8.2, U3.23 (DVDD), U3.45 (VREG_VOUT), U3.50 (DVDD)
- new net ADC3: J1.12 (Pin_12), U3.41 (GPIO29_ADC3)
- new net Button_2: C23.1, R15.2, U3.9 (GPIO7)
- new net Button_3: C24.1, R16.2, U3.12 (GPIO9)
- new net D: Q3.3 (G), R4.1, U3.11 (GPIO8)
- new net D_o: J2.7 (Pin_7), Q3.4 (D)
- new net E: Q1.1 (G), R5.1, U3.13 (GPIO10)
- new net E_o: J2.9 (Pin_9), Q1.6 (D)
- new net SCLK: U2.6 (CLK), U3.52 (QSPI_SCLK)
- new net SD0: U2.5 (DI(IO0)), U3.53 (QSPI_SD0)
- new net SD1: U2.2 (DO(IO1)), U3.55 (QSPI_SD1)
- new net SD2: U2.3 (IO2), U3.54 (QSPI_SD2)
- new net SD3: U2.7 (IO3), U3.51 (QSPI_SD3)
- new net SSel: JP1.2 (B), U2.1 (~{CS}), U3.56 (QSPI_SS)
- new net USB_D+: J7.2 (Pin_2), J8.3 (D+), R6.1
- new net USB_D-: J7.3 (Pin_3), J8.2 (D-), R7.1
- new net XIN: C21.1, U3.20 (XIN), Y1.3
- new net XOUT: R13.1, U3.21 (XOUT)
- no-connect marks 5 -> 13
Other:
- note added: "V2.0"
- note removed: "STM32L011F4 is pin-compatible"
- note removed: "Three channel LED drive. Intended to drive paralleled strings."
- moved on the sheet: C1, C18, C2, C22, C3, C4, H1, H2, H3, J3, J5, J6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
